File: schematic/sbc.sch (KiCad schematic (older format))
At the start: 5 parts

Commit message: sbc schematic update
Parts:
- added C?: .01uF, symbol C_Small
- added R? (x5): 3.3, symbol Rsqig
- added U?: 74LS08, symbol 74LS08
Connections:
- net labels added: +5v, CLOCK, GND, R~W~, ~IRQ1~, ~IRQ2~, ~IRQ~, ~RESET~
- wire segments 0 -> 26
- no-connect marks 0 -> 6
Other:
- note added: "remove 3.3k, \nand connect IRQ\nlater"
- moved on the sheet: U?
