File: schematic/IO.sch (KiCad schematic (older format))
At the start: 7 parts

Commit message: SBC Schematic final
Other:
- note added: "December 10th, 2016"
- note added: "Micheal Burin - ECEN 5613"
- note added: "SBC - I/O"
Changed lines of the file:
@@
 Wire Wire Line
 	2825 2225 2950 2225
+Text Notes 7025 6675 0    60   ~ 0
+Micheal Burin - ECEN 5613
+Text Notes 7400 7500 0    60   ~ 0
+SBC - I/O
+Text Notes 8150 7650 0    60   ~ 0
+December 10th, 2016
 $EndSCHEMATC
