File: schematic/power.sch (KiCad schematic (older format))
At the start: 12 parts

Commit message: SBC Schematic final
Other:
- note added: "December 10th, 2016"
- note added: "Micheal Burin - ECEN 5613"
- note added: "SBC - Power"
Changed lines of the file:
@@
 Wire Wire Line
 	4875 4650 4175 4650
+Text Notes 7050 6675 0    60   ~ 0
+Micheal Burin - ECEN 5613
+Text Notes 7400 7500 0    60   ~ 0
+SBC - Power
+Text Notes 8150 7650 0    60   ~ 0
+December 10th, 2016
 $EndSCHEMATC
